File: hw/characterizer/characterizer.kicad_pcb (KiCad board)
At the start: 2 copper layers, 229 parts, among them J1 1988820, J10 36-54-ND, J11 36-54-ND, J2 Conn_02x05_Odd_Even, J3 10118194-0001LF, J4 36-54-ND, J5 36-54-ND, J6 36-54-ND, J7 36-54-ND, J8 36-54-ND, J9 36-54-ND, Q1 BSS123, Q10 BSS123, Q11 FDMA008P20LZ, Q12 FDMA008P20LZ, Q13 BSS84, Q14 BSS123, Q15 BSS123, Q16 BSS123, Q17 FDMA008P20LZ, Q18 FDMA008P20LZ, Q19 PSMN7R0-30MLC,115, Q2 BSS123, Q20 BSS123, Q21 BSS84, Q22 BSS123, Q23 BSS123, Q24 BSS123, Q25 FDMA008P20LZ, Q26 FDMA008P20LZ, Q27 BSS84, Q28 BSS123, Q29 FDMA008P20LZ, Q3 FDMA008P20LZ, Q30 FDMA008P20LZ, Q31 FDMA008P20LZ, Q32 FDMA008P20LZ, Q33 FDMA008P20LZ, Q34 FDMA008P20LZ, Q35 FDMA008P20LZ, Q36 FDMA008P20LZ, Q4 FDMA008P20LZ, Q5 PSMN7R0-30MLC,115, Q6 BSS123, Q7 BSS84, Q8 BSS123, Q9 BSS123, U1 MIC5205-3.3, U10 AT30TS74, U11 TLV272CS-13, U12 TPS54719, U13 TLV272CS-13, U2 STM32F042K6T6, U3 74LVC2G04GW,125, U4 AT30TS74, U5 AT30TS74, U6 TLV272CS-13, U7 TPS54719, U8 TLV272CS-13, U9 AT30TS74, Y1 ABLS-8.000MHZ-B4-T

Commit message: layout functionally complete
Parts:
- removed TP1, TP10, TP11, TP12, TP2, TP3, TP4, TP5, TP6, TP7, TP8, TP9: Test_Point, Connector_PinHeader_2.54mm:PinHeader_1x01_P2.54mm_Vertical
- C34, C37, C38, C39, C40, C41, C42, C43, C44, C45, C46, C47, C48, L2, Q10, Q19, Q20, Q21, Q22, Q23, Q24, Q25, Q26, Q27, Q28, Q35, Q36, Q9, R46, R47, R73, R76, R77, R79, R80, R81, R82, R83, R84, R85, R86, R87, R88, R89, R90, R91, R92, R93, R94, R95, R96, R97, R98, U12, U13: moved to B.Cu
- moved C8 309.5 mm to (145.0, 85.5), turned to 180 degrees
- moved C6 309.1 mm to (145.1, 100.8), turned to 180 degrees
- moved Y1 305.5 mm to (145.4, 93.2), turned to 90 degrees
- moved Q10 299.9 mm to (172.8, 94.3), turned to 90 degrees
- moved R21 299.7 mm to (138.3, 84.0), turned to 180 degrees
- moved R19 299.6 mm to (138.3, 85.3), turned to 0 degrees
- moved C5 298.6 mm to (141.8, 90.8), turned to 90 degrees
- moved R13 297.1 mm to (138.3, 82.6), turned to 0 degrees
- moved R15 297.1 mm to (138.3, 81.2), turned to 180 degrees
- moved R47 296.6 mm to (172.3, 91.8), turned to 0 degrees
- moved R18 296.2 mm to (134.8, 101.0)
- moved R17 295.2 mm to (132.2, 85.2)
- moved Q9 295.1 mm to (181.6, 79.8)
- moved C12 294.9 mm to (133.1, 99.6), turned to 180 degrees
- moved C7 294.7 mm to (140.6, 96.5), turned to 180 degrees
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Connections:
- R15 pad 1: /mcu/VBAT1 -> /mcu/VBAT0
- R16 pad 1: /mcu/VBAT3 -> /mcu/VBAT2
- R21 pad 1: /mcu/VBAT0 -> /mcu/VBAT1
- R22 pad 1: /mcu/VBAT2 -> /mcu/VBAT3
- U3 pad 1: /pairA/DIR -> /pairB/DIR
- U3 pad 3: /pairB/DIR -> /pairA/DIR
- U3 pad 4: /pairB/nDIR -> /pairA/nDIR
- U3 pad 6: /pairA/nDIR -> /pairB/nDIR
Routing:
- net +6V: track 0.00 -> 500.2 mm, vias 0 -> 14
- net +3V3: track 0.00 -> 366.6 mm, vias 0 -> 10
- net GND: track 0.00 -> 315.5 mm, vias 0 -> 186
- net /mcu/VBAT1: track 0.00 -> 181.3 mm, vias 0 -> 2
- net /SCL: track 0.00 -> 146.9 mm, vias 0 -> 6
- net /mcu/VBAT0: track 0.00 -> 146.4 mm, vias 0 -> 1
- net /mcu/VBAT2: track 0.00 -> 144.1 mm, vias 0 -> 3
- net /SDA: track 0.00 -> 140.4 mm, vias 0 -> 6
- net /pairB/DIR: track 0.00 -> 131.5 mm, vias 0 -> 6
- net /mcu/VBAT3: track 0.00 -> 119.6 mm
- net /pairA/nDIR: track 0.00 -> 118.1 mm, vias 0 -> 3
- net /mcu/CEN_B: track 0.00 -> 115.4 mm, vias 0 -> 3
- net /pairA/DIR: track 0.00 -> 113.2 mm, vias 0 -> 4
- net /mcu/CC_A: track 0.00 -> 106.3 mm, vias 0 -> 3
- net /pairB/nDIR: track 0.00 -> 105.2 mm, vias 0 -> 4
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- added copper zone on B.Cu, net GND
- added copper zone on F.Cu, net GND
- added copper zone on In1.Cu, net GND
- added copper zone on B.Cu, net Net-(C17-Pad2)
- added copper zone on F.Cu, net Net-(C17-Pad2)
- added copper zone on B.Cu, net Net-(C34-Pad2)
- added copper zone on F.Cu, net Net-(C34-Pad2)
Other:
- copper layers 2 -> 4
- net class Default: clearance 0.26 -> 0.24; trace_width 0.26 -> 0.24; via_dia 0.64 -> 0.48; via_drill 0.4 -> 0.26
- net class bigger added: clearance 0.26, trace_width 0.28, via_dia 0.64, via_drill 0.42
- net class minimum removed
- rule trace_clearance: 0.26 -> 0.24
- rule trace_min: 0.127 -> 0.24

Commit message: layout as-ordered
Parts:
- moved C2 1.85 mm to (129.2, 130.2)
- moved C3 1.85 mm to (126.7, 129.6)
- moved R2 1.85 mm to (127.3, 137.3)
- moved R3 1.85 mm to (129.2, 133.1)
- moved U1 1.85 mm to (126.8, 132.3)
- moved C1 1.85 mm to (126.5, 135.1)
- moved R1 1.85 mm to (125.7, 137.3)
- moved Q2 1.23 mm to (156.8, 79.3)
- moved Q16 1.22 mm to (156.8, 121.1)
Routing:
- net GND: track 315.5 -> 312.8 mm, vias 186 -> 190
- net +3V3: track 366.6 -> 368.7 mm
- net /pairA/DIR: track 113.2 -> 115.1 mm
- net +6V: track 500.2 -> 498.3 mm
- net /pairB/DIR: track 131.5 -> 132.4 mm
- net /mcu/VBAT1: track 181.3 -> 180.5 mm
- net +5V: track 3.29 -> 4.07 mm
Other:
- board outline added: 113 x 93.7 mm
- board text added: "4x18650 characterizer v0.1 patrickyeon"
