File: hw/characterizer/characterizer.kicad_pcb (KiCad board)
At the start: 4 copper layers, 113 x 93.7 mm, 217 parts, among them J1 1988820, J10 36-54-ND, J11 36-54-ND, J2 Conn_02x05_Odd_Even, J3 10118194-0001LF, J4 36-54-ND, J5 36-54-ND, J6 36-54-ND, J7 36-54-ND, J8 36-54-ND, J9 36-54-ND, Q1 BSS123, Q10 BSS123, Q11 FDMA008P20LZ, Q12 FDMA008P20LZ, Q13 BSS84, Q14 BSS123, Q15 BSS123, Q16 BSS123, Q17 FDMA008P20LZ, Q18 FDMA008P20LZ, Q19 PSMN7R0-30MLC,115, Q2 BSS123, Q20 BSS123, Q21 BSS84, Q22 BSS123, Q23 BSS123, Q24 BSS123, Q25 FDMA008P20LZ, Q26 FDMA008P20LZ, Q27 BSS84, Q28 BSS123, Q29 FDMA008P20LZ, Q3 FDMA008P20LZ, Q30 FDMA008P20LZ, Q31 FDMA008P20LZ, Q32 FDMA008P20LZ, Q33 FDMA008P20LZ, Q34 FDMA008P20LZ, Q35 FDMA008P20LZ, Q36 FDMA008P20LZ, Q4 FDMA008P20LZ, Q5 PSMN7R0-30MLC,115, Q6 BSS123, Q7 BSS84, Q8 BSS123, Q9 BSS123, U1 MIC5205-3.3, U10 AT30TS74, U11 TLV272CS-13, U12 TPS54719, U13 TLV272CS-13, U2 STM32F042K6T6, U3 74LVC2G04GW,125, U4 AT30TS74, U5 AT30TS74, U6 TLV272CS-13, U7 TPS54719, U8 TLV272CS-13, U9 AT30TS74, Y1 ABLS-8.000MHZ-B4-T

Commit message: small board fixes
Parts:
- moved BT4 0.06 mm to (200.1, 111.6), turned to 180 degrees
- turned BT3 to 180 degrees
Other:
- board text added: "4x18650 characterizer v0.2 patrickyeon"
- board text removed: "4x18650 characterizer v0.1 patrickyeon"
Changed lines of the file:
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@@
   (layers
     (0 F.Cu signal)
-    (1 In1.Cu signal)
-    (2 In2.Cu signal)
-    (31 B.Cu signal)
-    (32 B.Adhes user)
-    (33 F.Adhes user)
-    (34 B.Paste user)
+    (1 In1.Cu signal hide)
+    (2 In2.Cu signal hide)
+    (31 B.Cu signal hide)
+    (32 B.Adhes user hide)
+    (33 F.Adhes user hide)
+    (34 B.Paste user hide)
     (35 F.Paste user)
-    (36 B.SilkS user)
+    (36 B.SilkS user hide)
     (37 F.SilkS user)
-    (38 B.Mask user)
+    (38 B.Mask user hide)
     (39 F.Mask user)
-    (40 Dwgs.User user)
-    (41 Cmts.User user)
-    (42 Eco1.User user)
-    (43 Eco2.User user)
+    (40 Dwgs.User user hide)
+    (41 Cmts.User user hide)
+    (42 Eco1.User user hide)
+    (43 Eco2.User user hide)
     (44 Edge.Cuts user)
-    (45 Margin user)
-    (46 B.CrtYd user)
+    (45 Margin user hide)
+    (46 B.CrtYd user hide)
     (47 F.CrtYd user)
-    (48 B.Fab user)
+    (48 B.Fab user hide)
     (49 F.Fab user)
   )
@@
   )
   (module project:18650-keyelco (layer F.Cu)
-    (at 184.37 132.5)
-    (fp_text reference BT3 (at 2.9 8.6) (layer F.SilkS) hide
+    (at 184.33 132.49 180)
+    (fp_text reference BT3 (at 2.9 8.6 180) (layer F.SilkS) hide
       (effects (font (size 1 1) (thickness 0.15)))
     )
-    (fp_text value Battery_Cell (at 0.6 -7.2) (layer F.Fab)
+    (fp_text value Battery_Cell (at 0.6 -7.2 180) (layer F.Fab)
       (effects (font (size 1 1) (thickness 0.15)))
     )
-    (fp_text user - (at -14.2 -0.5) (layer F.SilkS)
+    (fp_text user - (at -14.2 -0.5 180) (layer F.SilkS)
       (effects (font (size 7 7) (thickness 0.25)))
     )
@@
   )
   (module project:18650-keyelco (layer F.Cu)
-    (at 200.17 111.6)
-    (fp_text reference BT4 (at 2.9 8.6) (layer F.SilkS) hide
+    (at 200.13 111.56 180)
+    (fp_text reference BT4 (at 2.9 8.6 180) (layer F.SilkS) hide
       (effects (font (size 1 1) (thickness 0.15)))
     )
-    (fp_text value Battery_Cell (at 0.6 -7.2) (layer F.Fab)
+    (fp_text value Battery_Cell (at 0.6 -7.2 180) (layer F.Fab)
       (effects (font (size 1 1) (thickness 0.15)))
     )
@@
     (fp_circle (center 23.5 -2.54) (end 22 -2.54) (layer F.SilkS) (width 0.15))
     (fp_circle (center -23.5 -2.54) (end -25 -2.54) (layer F.SilkS) (width 0.15))
-    (fp_text user + (at 14 -0.4) (layer F.SilkS)
+    (fp_text user + (at 14 -0.4 180) (layer F.SilkS)
       (effects (font (size 7 7) (thickness 0.25)))
     )
-    (fp_text user - (at -14.2 -0.5) (layer F.SilkS)
+    (fp_text user - (at -14.2 -0.5 180) (layer F.SilkS)
       (effects (font (size 7 7) (thickness 0.25)))
     )
@@
   (gr_line (start 150.675 115.625) (end 146.075 115.625) (layer F.SilkS) (width 0.1))
   (gr_line (start 151.35 114.95) (end 150.675 115.625) (layer F.SilkS) (width 0.1))
-  (gr_text "4x18650 characterizer  v0.1\npatrickyeon" (at 134.975 57.15) (layer F.SilkS)
+  (gr_text "4x18650 characterizer  v0.2\npatrickyeon" (at 134.975 57.15) (layer F.SilkS)
     (effects (font (size 3 3) (thickness 0.5)) (justify left))
   )
@@
   (gr_line (start 146.2 74) (end 150.5 74) (layer F.SilkS) (width 0.2))
   (gr_line (start 146.2 71.5) (end 146.2 74) (layer F.SilkS) (width 0.2))
-  (via (at 126.7 142) (size 3.8) (drill 3.4) (layers F.Cu B.Cu) (net 2))
-  (via (at 232.3 55.7) (size 3.8) (drill 3.4) (layers F.Cu B.Cu) (net 2))
-  (via (at 126.7 55.7) (size 3.8) (drill 3.4) (layers F.Cu B.Cu) (net 2))
-  (via (at 232.3 142) (size 3.8) (drill 3.4) (layers F.Cu B.Cu) (net 2))
   (segment (start 125.75 135.1125) (end 125.7625 135.1) (width 0.25) (layer F.Cu) (net 1))
   (segment (start 125.75 136.5125) (end 125.75 135.1125) (width 0.25) (layer F.Cu) (net 1))
@@
   (segment (start 126.12 132.3) (end 126.1325 132.3125) (width 0.25) (layer F.Cu) (net 1))
   (segment (start 125.75 136.5125) (end 127.35 136.5125) (width 0.25) (layer F.Cu) (net 1))
+  (via (at 126.7 142) (size 3.8) (drill 3.4) (layers F.Cu B.Cu) (net 2))
+  (via (at 232.3 55.7) (size 3.8) (drill 3.4) (layers F.Cu B.Cu) (net 2))
+  (via (at 126.7 55.7) (size 3.8) (drill 3.4) (layers F.Cu B.Cu) (net 2))
+  (via (at 232.3 142) (size 3.8) (drill 3.4) (layers F.Cu B.Cu) (net 2))
   (segment (start 185.07 132.35) (end 184.2325 132.35) (width 0.25) (layer B.Cu) (net 2))
   (segment (start 184.2325 132.35) (end 184.17 132.2875) (width 0.25) (layer B.Cu) (net 2))
