File: hw/characterizer/control.sch (KiCad schematic (older format))
At the start: 35 parts, among them J2 Conn_02x05_Odd_Even, J3 10118194-0001LF, U2 STM32F042K6T6, U3 74LVC2G04GW,125, Y1 ABLS-8.000MHZ-B4-T

Commit message: layout functionally complete
Changed lines of the file:
@@
 Text HLabel 7000 3250 2    50   Input ~ 0
 DC_B
+Text HLabel 6550 3550 2    50   Input ~ 0
+VBAT0
 Text HLabel 7300 3400 2    50   Input ~ 0
-VBAT0
-Text HLabel 6550 3550 2    50   Input ~ 0
 VBAT1
 Text HLabel 7050 2000 2    50   Output ~ 0
@@
 $EndComp
 Connection ~ 5200 1550
+Text HLabel 6550 4400 2    50   Input ~ 0
+VBAT2
 Text HLabel 7300 4250 2    50   Input ~ 0
-VBAT2
-Text HLabel 6550 4400 2    50   Input ~ 0
 VBAT3
 $Comp
@@
 Wire Wire Line
 	5550 3650 5450 3650
+Text Label 4800 6300 0    50   ~ 0
+DIR_A
 Text Label 4800 6200 0    50   ~ 0
-DIR_A
-Text Label 4800 6300 0    50   ~ 0
 DIR_B
+Text HLabel 5850 6200 2    50   Output ~ 0
+nDIR_B
 Text HLabel 5850 6300 2    50   Output ~ 0
-nDIR_B
-Text HLabel 5850 6200 2    50   Output ~ 0
 nDIR_A
 Wire Wire Line

Commit message: updating schematic with digikey pns
Parts:
- J2: Digikey PN (none) -> 1175-1629-ND
- U2: Digikey PN (none) -> 497-14647-ND
- U3: Digikey PN (none) -> 1727-4032-1-ND
Changed lines of the file:
@@
 F 2 "project:CONN_JTAG_10" H 2350 2850 50  0001 C CNN
 F 3 "~" H 2350 2850 50  0001 C CNN
+F 4 "1175-1629-ND" H 0   0   50  0001 C CNN "Digikey PN"
 	1    2350 2850
 	1    0    0    -1
@@
 F 2 "Package_QFP:LQFP-32_7x7mm_P0.8mm" H 4350 2750 60  0001 C CNN
 F 3 "" H 4350 2750 60  0001 C CNN
+F 4 "497-14647-ND" H 0   0   50  0001 C CNN "Digikey PN"
 	1    4950 3150
 	1    0    0    -1
@@
 F 2 "Package_TO_SOT_SMD:SOT-363_SC-70-6" H 5350 6200 50  0001 C CNN
 F 3 "" H 5350 6200 50  0001 C CNN
+F 4 "1727-4032-1-ND" H 0   0   50  0001 C CNN "Digikey PN"
 	1    5350 6200
 	1    0    0    -1
