File: hw/characterizer/charger.sch (KiCad schematic (older format))
At the start: 44 parts, among them Q10 BSS123, Q11 FDMA008P20LZ, Q12 FDMA008P20LZ, Q13 BSS84, Q14 BSS123, Q31 FDMA008P20LZ, Q32 FDMA008P20LZ, Q9 BSS123, U7 TPS54719, U8 TLV272CS-13

Commit message: updating schematic with digikey pns
Parts:
- C21, C22, C23, C28: DK pn 311-1376-1-ND -> (none); Digikey PN (none) -> 311-1376-1-ND
- C29, C31: DK pn 311-1376-1-ND -> (none)
- L1: DK pn 495-1799-1-ND -> (none); Digikey PN (none) -> 495-1799-1-ND
- U7: Digikey PN (none) -> 296-36812-1-ND
- U8: Digikey PN (none) -> TLV272CS-13DICT-ND

Commit message: small board fixes
Parts:
- U8: Digikey PN TLV272CS-13DICT-ND -> TLV272IM8-13DICT-ND

Commit message: updated schematics with all the mods so far
Parts:
- removed C30: 100n, Capacitor_SMD:C_0603_1608Metric, symbol Device:C_Small
- removed C31: DNI, Capacitor_SMD:C_0603_1608Metric, symbol Device:C_Small
- removed R49, R55: 20k, Resistor_SMD:R_0603_1608Metric, symbol Device:R_Small
- removed R50, R52: 3k3, Resistor_SMD:R_0603_1608Metric, symbol Device:R_Small
- removed R57: 2k, Resistor_SMD:R_0603_1608Metric, symbol Device:R_Small
- removed R58: 1k, Resistor_SMD:R_0603_1608Metric, symbol Device:R_Small
- removed TP4, TP5, TP6: Test_Point, Connector_PinHeader_2.54mm:PinHeader_1x01_P2.54mm_Vertical, symbol Connector:Test_Point
- removed U8: TLV272CS-13, Package_SO:MSOP-8_3x3mm_P0.65mm, symbol Device:Opamp_Dual_Generic
- added C?: 1n, Capacitor_SMD:C_0603_1608Metric, symbol Device:C_Small
- added C?: 10n, Capacitor_SMD:C_0603_1608Metric, symbol Device:C_Small
- added C?: 100n, Capacitor_SMD:C_0603_1608Metric, symbol Device:C_Small
- added D? (x2): 1N4148, Diode_THT:D_DO-35_SOD27_P7.62mm_Horizontal, symbol Diode:1N4148
- added R? (x6): 1k, Resistor_SMD:R_0603_1608Metric, symbol Device:R_Small
- added R? (x2): 2k, Resistor_SMD:R_0603_1608Metric, symbol Device:R_Small
- added R? (x2): 10k, Resistor_SMD:R_0603_1608Metric, symbol Device:R_Small
- added R? (x2): 250k, Resistor_SMD:R_0603_1608Metric, symbol Device:R_Small
- added R? (x2): 3k3, Resistor_SMD:R_0603_1608Metric, symbol Device:R_Small
- added U? (x5): TLV274, symbol Device:Opamp_Quad_Generic
- C29: value DNI -> 100n
- R59: value 0 -> 1k
Connections:
- wire segments 139 -> 175
Other:
- note added: "TODO: whatever diode makes sense"
