File: hw/characterizer/load.sch (KiCad schematic (older format))
At the start: 32 parts, among them Q1 BSS123, Q2 BSS123, Q29 FDMA008P20LZ, Q3 FDMA008P20LZ, Q30 FDMA008P20LZ, Q4 FDMA008P20LZ, Q5 PSMN7R0-30MLC,115, Q6 BSS123, Q7 BSS84, Q8 BSS123, U6 TLV272CS-13

Commit message: updating schematic with digikey pns
Parts:
- U6: Digikey PN (none) -> TLV272CS-13DICT-ND
Changed lines of the file:
@@
 F 2 "Package_SO:MSOP-8_3x3mm_P0.65mm" H 6100 2950 50  0001 C CNN
 F 3 "~" H 6100 2950 50  0001 C CNN
+F 4 "TLV272CS-13DICT-ND" H 0   0   50  0001 C CNN "Digikey PN"
 	1    6100 2950
 	1    0    0    -1
@@
 F 2 "Package_SO:MSOP-8_3x3mm_P0.65mm" H 7700 3300 50  0001 C CNN
 F 3 "~" H 7700 3300 50  0001 C CNN
+F 4 "TLV272CS-13DICT-ND" H 0   0   50  0001 C CNN "Digikey PN"
 	2    7700 3300
 	1    0    0    -1
@@
 F 2 "Package_SO:MSOP-8_3x3mm_P0.65mm" H 7700 3300 50  0001 C CNN
 F 3 "~" H 7700 3300 50  0001 C CNN
+F 4 "TLV272CS-13DICT-ND" H 0   0   50  0001 C CNN "Digikey PN"
 	3    7700 3300
 	1    0    0    -1

Commit message: small board fixes
Parts:
- U6: Digikey PN TLV272CS-13DICT-ND -> TLV272IM8-13DICT-ND

Commit message: updated schematics with all the mods so far
Parts:
- removed C18: 100n, Capacitor_SMD:C_0603_1608Metric, symbol Device:C_Small
- removed C19: DNI, Capacitor_SMD:C_0603_1608Metric, symbol Device:C_Small
- removed Q7: BSS84, Package_TO_SOT_SMD:SOT-23, symbol Device:Q_PMOS_GSD
- removed R31, R35: 20k, Resistor_SMD:R_0603_1608Metric, symbol Device:R_Small
- removed R32, R34: 3k3, Resistor_SMD:R_0603_1608Metric, symbol Device:R_Small
- removed R37: 2k, Resistor_SMD:R_0603_1608Metric, symbol Device:R_Small
- removed R38, R41: 1k, Resistor_SMD:R_0603_1608Metric, symbol Device:R_Small
- removed R42: 10k, Resistor_SMD:R_0603_1608Metric, symbol Device:R_Small
- removed TP1, TP2, TP3: Test_Point, Connector_PinHeader_2.54mm:PinHeader_1x01_P2.54mm_Vertical, symbol Connector:Test_Point
- removed U6: TLV272CS-13, Package_SO:MSOP-8_3x3mm_P0.65mm, symbol Device:Opamp_Dual_Generic
- added C?: 10n, Capacitor_SMD:C_0603_1608Metric, symbol Device:C_Small
- added C?: 100n, Capacitor_SMD:C_0603_1608Metric, symbol Device:C_Small
- added D? (x2): 1N4148, Diode_THT:D_DO-35_SOD27_P7.62mm_Horizontal, symbol Diode:1N4148
- added Q?: BSS123, Package_TO_SOT_SMD:SOT-23, symbol Device:Q_NMOS_GSD
- added R? (x5): 1k, Resistor_SMD:R_0603_1608Metric, symbol Device:R_Small
- added R? (x2): 2k, Resistor_SMD:R_0603_1608Metric, symbol Device:R_Small
- added R? (x3): 10k, Resistor_SMD:R_0603_1608Metric, symbol Device:R_Small
- added R? (x2): 250k, Resistor_SMD:R_0603_1608Metric, symbol Device:R_Small
- added R? (x2): 3k3, Resistor_SMD:R_0603_1608Metric, symbol Device:R_Small
- added R?: 1M, Resistor_SMD:R_0603_1608Metric, symbol Device:R_Small
- added U? (x5): TLV274, symbol Device:Opamp_Quad_Generic
- C17: value DNI -> 10n
- R36: value 3k3 -> 10k
Connections:
- wire segments 96 -> 130
