File: hw/characterizer/pair.sch (KiCad schematic (older format))
At the start: 16 parts, among them J4 36-54-ND, J5 36-54-ND, J6 36-54-ND, J7 36-54-ND, U4 AT30TS74, U5 AT30TS74

Commit message: updating schematic with digikey pns
Parts:
- J4, J5, J6, J7: Digikey PN (none) -> 36-54-ND
Changed lines of the file:
@@
 F 2 "project:BATTERY_CLIP_36-54" H 4500 6600 50  0001 C CNN
 F 3 "~" H 4500 6600 50  0001 C CNN
+F 4 "36-54-ND" H 0   0   50  0001 C CNN "Digikey PN"
 	1    4500 6600
 	0    1    1    0
@@
 F 2 "project:BATTERY_CLIP_36-54" H 4500 5650 50  0001 C CNN
 F 3 "~" H 4500 5650 50  0001 C CNN
+F 4 "36-54-ND" H 0   0   50  0001 C CNN "Digikey PN"
 	1    4500 5650
 	0    -1   -1   0
@@
 F 2 "project:BATTERY_CLIP_36-54" H 4350 3400 50  0001 C CNN
 F 3 "~" H 4350 3400 50  0001 C CNN
+F 4 "36-54-ND" H 0   0   50  0001 C CNN "Digikey PN"
 	1    4350 3400
 	0    1    1    0
@@
 F 2 "project:BATTERY_CLIP_36-54" H 4350 2450 50  0001 C CNN
 F 3 "~" H 4350 2450 50  0001 C CNN
+F 4 "36-54-ND" H 0   0   50  0001 C CNN "Digikey PN"
 	1    4350 2450
 	0    -1   -1   0
